Commit message: minor changes, mainlny KITTY alignments

File: launch/include/config/robot.urdf.xacro (robot description, xacro)
@@ -15,4 +15,10 @@
     <origin xyz="0 0 0" rpy="0 0 0" />
   </joint>
+  <link name="imu_enu_link"> </link>
+  <joint name="imu_enu_joint" type="fixed">
+    <parent link="chassis_link" />
+    <child link="imu_enu_link" />
+    <origin xyz="0 0 0" rpy="0 0 0" />
+  </joint>
   <link name="velodyne"> </link>
   <joint name="velodyne_joint" type="fixed">
